File: hardware/v2/esp32-adapter-board/esp32-adapter-board.kicad_pcb (KiCad board)
At the start: 2 copper layers, 80 x 30 mm, 6 parts

Commit message: Add v2 hardware updates: gerber files, updated KiCad projects, schematic revisions
Co-Authored-By: Claude Sonnet 4.6 <noreply@anthropic.com>
Parts:
- ESP32 DEVKITC: renamed from ESP32 Wroom-32D
Routing:
- net Net-(J33-Pin_3): track 25.4 -> 42.9 mm
- net Net-(J33-Pin_12): track 55.3 -> 44.0 mm
- net Net-(J33-Pin_2): track 27.3 -> 36.6 mm
- net Net-(J33-Pin_10): track 48.6 -> 40.4 mm
- net Net-(J33-Pin_4): track 40.7 -> 45.3 mm
- net Net-(J33-Pin_8): track 51.2 -> 47.6 mm, vias 1 -> 0
- net Net-(J33-Pin_5): track 50.2 -> 48.6 mm
- net Net-(J33-Pin_11): track 36.6 -> 35.3 mm
- net Net-(J33-Pin_7): track 52.0 -> 53.2 mm
- net Net-(J33-Pin_6): track 46.0 -> 45.5 mm, vias 0 -> 1
- net Net-(J33-Pin_16): vias 1 -> 0
- net Net-(J33-Pin_14): vias 1 -> 0
Other:
- board text added: "ESP32 Adapter-Board 1 2026 - bigbrainlabs"
