File: hardware/v2/input-board/input-board.kicad_pcb (KiCad board)
At the start: 2 copper layers, 110 x 46 mm, 30 parts, among them J27 Screw_Terminal_01x16

Commit message: Add v2 hardware updates: gerber files, updated KiCad projects, schematic revisions
Co-Authored-By: Claude Sonnet 4.6 <noreply@anthropic.com>
Routing:
- net GND: track 8.48 -> 11.0 mm, vias 6 -> 8
Other:
- board text added: "16 Channel Input-Board 2026 - bigbrainlabs"
Changed lines of the file:
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@@
 			(outputformat 1)
 			(mirror no)
-			(drillshape 1)
+			(drillshape 0)
 			(scaleselection 1)
-			(outputdirectory "")
+			(outputdirectory "gerber/")
 		)
 	)
@@
 		(layer "Edge.Cuts")
 	)
+	(gr_text "16 Channel Input-Board\n2026 - bigbrainlabs"
+		(at 173.5 84 0)
+		(layer "F.SilkS")
+		(effects
+			(font
+				(size 1 1)
+				(thickness 0.1)
+			)
+			(justify left)
+		)
+	)
 	(gr_text "(Bourns 4116R-1-102LF), DIP-16, isolated."
 		(at 169 75.5 0)
@@
 		(net 33)
 	)
+	(segment
+		(start 168 83)
+		(end 168 85.5)
+		(width 0.2)
+		(layer "F.Cu")
+		(net 33)
+	)
 	(via
 		(at 122.1773 72.5922)
@@
 	)
 	(via
+		(at 168 85.5)
+		(size 0.6)
+		(drill 0.3)
+		(layers "F.Cu" "B.Cu")
+		(free yes)
+		(net 33)
+	)
+	(via
 		(at 113.9426 72.6363)
 		(size 0.6)
@@
 		(net 33)
 	)
+	(via
+		(at 168 83)
+		(size 0.6)
+		(drill 0.3)
+		(layers "F.Cu" "B.Cu")
+		(free yes)
+		(net 33)
+	)
