File: hardware/v2/input-board/input-board.kicad_sch (KiCad schematic)
At the start: 0 parts

Commit message: Hardware v2: Input-Board neu generiert (Rev.1/Rev.2)
Gerber neu erzeugt, rev1/rev2-ZIP und Pick-&-Place-CSV ergänzt,
Schaltplan/Layout und Projektdateien aktualisiert.

Co-Authored-By: Claude Opus 4.8 <noreply@anthropic.com>
Parts:
- added D1, D10, D11, D12, D13, D14, D15, D16, D2, D3, D4, D5, D6, D7, D8, D9: D_Zener, PCM_Diode_SMD_AKL:D_SOD-123_Zener, symbol Device:D_Zener
- added J1, J10, J11, J12, J13, J14, J15, J16, J2, J3, J4, J5, J6, J7, J8, J9: Conn_01x03_Pin, Connector_JST:JST_PH_B3B-PH-K_1x03_P2.00mm_Vertical, symbol Connector:Conn_01x03_Pin
- added J27: Screw_Terminal_01x16, TerminalBlock_Phoenix:TerminalBlock_Phoenix_MKDS-3-16-5.08_1x16_P5.08mm_Horizontal, symbol Connector:Screw_Terminal_01x16
- added J29: Conn_02x10_Odd_Even, Connector_PinHeader_2.54mm:PinHeader_2x10_P2.54mm_Vertical, symbol Connector_Generic:Conn_02x10_Odd_Even
- added R1, R10, R11, R12, R13, R14, R15, R16, R2, R3, R4, R5, R6, R7, R8, R9: 1k, Resistor_SMD:R_0805_2012Metric, symbol PCM_SL_Resistors:1k
- added R17, R18, R19, R20, R21, R22, R23, R24, R25, R26, R27, R28, R29, R30, R31, R32: 1M, Resistor_SMD:R_0805_2012Metric, symbol PCM_SL_Resistors:1M
Connections:
- new net: J27.6 (Pin_6), J6.1 (Pin_1)
- new net: J6.3 (Pin_3), R6.2
- new net: D1.1 (K), J29.1 (Pin_1), R1.1, R17.1
- new net: D10.1 (K), J29.10 (Pin_10), R10.1, R26.1
- new net: D11.1 (K), J29.11 (Pin_11), R11.1, R27.1
- new net: D12.1 (K), J29.12 (Pin_12), R12.1, R28.1
- new net: D13.1 (K), J29.13 (Pin_13), R13.1, R29.1
- new net: D14.1 (K), J29.14 (Pin_14), R14.1, R30.1
- new net: D15.1 (K), J29.15 (Pin_15), R15.1, R31.1
- new net: D16.1 (K), J29.16 (Pin_16), R16.1, R32.1
- new net: D2.1 (K), J29.2 (Pin_2), R18.1, R2.1
- new net: D3.1 (K), J29.3 (Pin_3), R19.1, R3.1
- new net: D4.1 (K), J29.4 (Pin_4), R20.1, R4.1
- new net: D5.1 (K), J29.5 (Pin_5), R21.1, R5.1
- new net: D6.1 (K), J29.6 (Pin_6), R22.1, R6.1
- new net: D7.1 (K), J29.7 (Pin_7), R23.1, R7.1
- new net: D8.1 (K), J29.8 (Pin_8), R24.1, R8.1
- new net: D9.1 (K), J29.9 (Pin_9), R25.1, R9.1
- new net: J4.3 (Pin_3), R4.2
- new net: J14.3 (Pin_3), R14.2
- new net: J3.3 (Pin_3), R3.2
- new net: J27.8 (Pin_8), J8.1 (Pin_1)
- new net: J8.3 (Pin_3), R8.2
- new net: J10.3 (Pin_3), R10.2
- new net: J1.1 (Pin_1), J27.1 (Pin_1)
- new net: J1.3 (Pin_3), R1.2
- new net: J27.7 (Pin_7), J7.1 (Pin_1)
- new net: J7.3 (Pin_3), R7.2
- new net: J15.1 (Pin_1), J27.15 (Pin_15)
- new net: J15.3 (Pin_3), R15.2
- new net: J10.1 (Pin_1), J27.10 (Pin_10)
- new net: J11.1 (Pin_1), J27.11 (Pin_11)
- new net: J11.3 (Pin_3), R11.2
- new net: J16.3 (Pin_3), R16.2
- new net: J27.5 (Pin_5), J5.1 (Pin_1)
- new net: J5.3 (Pin_3), R5.2
- new net: J12.3 (Pin_3), R12.2
- new net: J27.9 (Pin_9), J9.1 (Pin_1)
- new net: J9.3 (Pin_3), R9.2
- new net: J14.1 (Pin_1), J27.14 (Pin_14)
- new net: J2.1 (Pin_1), J27.2 (Pin_2)
- new net: J2.3 (Pin_3), R2.2
- new net: J12.1 (Pin_1), J27.12 (Pin_12)
- new net: J13.1 (Pin_1), J27.13 (Pin_13)
- new net: J13.3 (Pin_3), R13.2
- new net: J27.4 (Pin_4), J4.1 (Pin_1)
- new net: J27.3 (Pin_3), J3.1 (Pin_1)
- new net: J16.1 (Pin_1), J27.16 (Pin_16)
- new net GND: D1.2 (A), D10.2 (A), D11.2 (A), D12.2 (A), D13.2 (A), D14.2 (A), D15.2 (A), D16.2 (A), D2.2 (A), D3.2 (A), D4.2 (A), D5.2 (A), D6.2 (A), D7.2 (A), D8.2 (A), D9.2 (A), J1.2 (Pin_2), J10.2 (Pin_2), J11.2 (Pin_2), J12.2 (Pin_2), J13.2 (Pin_2), J14.2 (Pin_2), J15.2 (Pin_2), J16.2 (Pin_2), J2.2 (Pin_2), J29.20 (Pin_20), J3.2 (Pin_2), J4.2 (Pin_2), J5.2 (Pin_2), J6.2 (Pin_2), J7.2 (Pin_2), J8.2 (Pin_2), J9.2 (Pin_2), R17.2, R18.2, R19.2, R20.2, R21.2, R22.2, R23.2, R24.2, R25.2, R26.2, R27.2, R28.2, R29.2, R30.2, R31.2, R32.2
- no-connect marks 0 -> 3
