File: hardware/v2/vcc-board/vcc-board.kicad_pcb (KiCad board)
At the start: 2 copper layers, 20 x 80 mm, 13 parts

Commit message: Add v2 hardware updates: gerber files, updated KiCad projects, schematic revisions
Co-Authored-By: Claude Sonnet 4.6 <noreply@anthropic.com>
Other:
- board text added: "VCC Borad 2026 - bigbrainlabs"
Changed lines of the file:
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@@
 			(outputformat 1)
 			(mirror no)
-			(drillshape 1)
+			(drillshape 0)
 			(scaleselection 1)
-			(outputdirectory "")
+			(outputdirectory "gerber/")
 		)
 	)
@@
 		)
 	)
+	(gr_text "VCC Borad \n2026 - bigbrainlabs"
+		(at 162.5 64.5 90)
+		(layer "F.SilkS")
+		(effects
+			(font
+				(size 1 1)
+				(thickness 0.1)
+			)
+			(justify left)
+		)
+	)
