File: hardware/v2/vcc-board/vcc-board.kicad_pcb (KiCad board)
At the start: 2 copper layers, 20 x 80 mm, 13 parts

Commit message: Hardware: VCC-Board Gerber/KiCad aktualisiert + MotorCombo THT Gehaeuse V1
- vcc-board: Gerber, Drill, KiCad-PCB/PRL aktualisiert (Silkscreen u.a.)
- MotorCombo THT: Gehaeuse V1 (3mf + STL Body/Lid) hinzugefuegt

Co-Authored-By: Claude Opus 4.8 <noreply@anthropic.com>
Other:
- board text added: "sponsored by"
